Commit message: urdf: lower the table buffer dimensions
Greetings didn't work once with the old values. There was a slight collision

Signed-off-by: Wolfgang Wiedmeyer <wolfgang.wiedmeyer@kit.edu>

File: urdf/playground_env.urdf.xacro (robot description, xacro)
@@ -18,14 +18,14 @@
     </inertial>
     <visual>
-      <origin xyz="0 0 0.09" rpy="0 0 0"/>
+      <origin xyz="0 0 0.08" rpy="0 0 0"/>
       <geometry>
-        <box size="1.2 1.6 0.18"/>
+        <box size="1.2 1.6 0.16"/>
       </geometry>
       <material name="transparent" />
     </visual>
     <collision>
-      <origin xyz="0 0 0.09" rpy="0 0 0"/>
+      <origin xyz="0 0 0.08" rpy="0 0 0"/>
       <geometry>
-        <box size="1.2 1.6 0.18"/>
+        <box size="1.2 1.6 0.16"/>
       </geometry>
     </collision>
