Commit message: Use the cap endeffector
Configured the project to use the new "cap" eef type instead of the gripper. The example code has been updated to reflect this change. The RViz config has been updated as well to show the correct cap TF. To better see what the project looks like a screenshot has been added to the Readme.

File: config/playground_cell.srdf.xacro (robot description, xacro)
@@ -2,6 +2,7 @@
 <robot xmlns:xacro="http://www.ros.org/wiki/xacro" name="rll_cell">
   <xacro:include filename="$(find rll_moveit_config)/config/rll_cell.xacro" />
-  <xacro:arg name="robot_name" default="iiwa"/>
-  <xacro:rll_cell robot_name="$(arg robot_name)"/>
+  <xacro:arg name="robot_name" default="iiwa" />
+  <xacro:arg name="eef_type" default="cap" />
+  <xacro:rll_cell robot_name="$(arg robot_name)" eef_type="$(arg eef_type)" />
   <disable_collisions link1="axis_cam_base" link2="table_buffer" reason="Never" />
   <disable_collisions link1="axis_cam_top" link2="table_buffer" reason="Never" />

File: urdf/playground_env.urdf.xacro (robot description, xacro)
@@ -1,31 +1,32 @@
 <?xml version="1.0"?>
 <robot xmlns:xacro="http://www.ros.org/wiki/xacro" name="rll_cell">
-  <xacro:include filename="$(find rll_description)/urdf/rll_cell.xacro"/>
-  <xacro:arg name="hardware_interface" default="PositionJointInterface"/>
-  <xacro:arg name="robot_name" default="iiwa"/>
-  <xacro:rll_cell hardware_interface="$(arg hardware_interface)" robot_name="$(arg robot_name)"/>
+  <xacro:include filename="$(find rll_description)/urdf/rll_cell.xacro" />
+  <xacro:arg name="hardware_interface" default="PositionJointInterface" />
+  <xacro:arg name="robot_name" default="iiwa" />
+  <xacro:arg name="eef_type" default="cap" />
+  <xacro:rll_cell hardware_interface="$(arg hardware_interface)" robot_name="$(arg robot_name)" eef_type="$(arg eef_type)" />
   <!-- This ensures that the robot cannot move close to the table -->
   <joint name="table_buffer" type="fixed">
     <parent link="world" />
     <child link="table_buffer" />
-    <origin xyz="0 0 0" rpy="0 0 0"/>
+    <origin xyz="0 0 0" rpy="0 0 0" />
   </joint>
   <link name="table_buffer">
     <inertial>
-      <origin xyz="0 0 0" rpy="0 0 0"/>
-      <mass value="1"/>
-      <inertia ixx="1" ixy="0" ixz="0" iyy="1" iyz="0" izz="1"/>
+      <origin xyz="0 0 0" rpy="0 0 0" />
+      <mass value="1" />
+      <inertia ixx="1" ixy="0" ixz="0" iyy="1" iyz="0" izz="1" />
     </inertial>
     <visual>
-      <origin xyz="0 0 0.08" rpy="0 0 0"/>
+      <origin xyz="0 0 0.08" rpy="0 0 0" />
       <geometry>
-        <box size="1.2 1.6 0.16"/>
+        <box size="1.2 1.6 0.16" />
       </geometry>
       <material name="transparent" />
     </visual>
     <collision>
-      <origin xyz="0 0 0.08" rpy="0 0 0"/>
+      <origin xyz="0 0 0.08" rpy="0 0 0" />
       <geometry>
-        <box size="1.2 1.6 0.16"/>
+        <box size="1.2 1.6 0.16" />
       </geometry>
     </collision>

Commit message: Tests: run playground.py in CI
Add a TestCase to run the playground.py via the CI. The lauch scripts have been adjusted to allow passing the use_sim parameter to specify whether or not to launch the script with Gazebo. The CI runs the script twice once with and once without gazebo. However, the gazebo-enabled version does seem to cause deviation errors from time to time.

File: config/playground_cell.srdf.xacro (robot description, xacro)
@@ -1,8 +1,8 @@
 <?xml version='1.0' encoding='utf-8'?>
 <robot xmlns:xacro="http://www.ros.org/wiki/xacro" name="rll_cell">
+  <xacro:arg name="robot_name" default="iiwa"/>
+  <xacro:arg name="eef_type" default="cap"/>
   <xacro:include filename="$(find rll_moveit_config)/config/rll_cell.xacro" />
-  <xacro:arg name="robot_name" default="iiwa" />
-  <xacro:arg name="eef_type" default="cap" />
-  <xacro:rll_cell robot_name="$(arg robot_name)" eef_type="$(arg eef_type)" />
+  <xacro:rll_cell robot_name="$(arg robot_name)" eef_type="$(arg eef_type)"/>
   <disable_collisions link1="axis_cam_base" link2="table_buffer" reason="Never" />
   <disable_collisions link1="axis_cam_top" link2="table_buffer" reason="Never" />

File: urdf/playground_env.urdf.xacro (robot description, xacro)
@@ -8,5 +8,5 @@
   <!-- This ensures that the robot cannot move close to the table -->
   <joint name="table_buffer" type="fixed">
-    <parent link="world" />
+    <parent link="table" />
     <child link="table_buffer" />
     <origin xyz="0 0 0" rpy="0 0 0" />
